File: _autosave-fast_respect.kicad_pcb (KiCad board)
At the start: 2 copper layers, 70 x 110 mm, 97 parts, among them J1_1 Conn_02x04_Odd_Even, J5_1 Conn_02x03_Odd_Even, J5_2 Conn_02x03_Odd_Even, J7_1 Conn_01x02, Q2_1 IRLML6402, Q3_1 IRLML6344T, Q4_1 IRLML6344T, Q4_2 IRLML6344T, Q4_3 IRLML6344T, Q4_4 IRLML6344T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

Commit message: 2sBatteryのフットプリント作成
Parts:
- moved R3_3 79.2 mm to (-7.42, 97.2)
- moved R3_4 78.4 mm to (-7.52, 95.1)
- moved R3_5 77.9 mm to (-7.62, 93.3)
- moved R3_6 77.8 mm to (-7.58, 91.3)
- moved R3_7 66.8 mm to (-18.6, 93.8), turned to 90 degrees
- moved R3_8 66.3 mm to (-19.1, 98.0), turned to 90 degrees
- moved Q3_1 64.7 mm to (-16.1, 101.1)
- moved U5_1 43.5 mm to (-46.4, 69.4), turned to 90 degrees
- moved R2_4 39.6 mm to (-66.9, 93.8)
- moved R2_3 39.0 mm to (-48.5, 93.0)
- moved R2_5 38.2 mm to (-62.8, 93.9)
- moved R2_2 34.0 mm to (-48.5, 95.8)
- moved BZ3_1 4.41 mm to (-14.0, 95.3)
- moved Q2_1 3.01 mm to (-53.4, 94.3)
- moved R2_1 2.45 mm to (-53.8, 98.4)
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
Commit message: バッテリ端子のフットプリントを割り当ててネットリストに出力して取り込み
Parts:
- BT2_1: footprint Connector_JST:JST_PH_B2B-PH-K_1x02_P2.00mm_Vertical -> Self-Made_Generic_Packages:2sBattery
Changed lines of the file:
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@@
     )
   )
-  (footprint "Connector_JST:JST_PH_B2B-PH-K_1x02_P2.00mm_Vertical" (layer "F.Cu")
+  (footprint "Self-Made_Generic_Packages:2sBattery" (layer "F.Cu")
     (at -47.88 103.71)
-    (descr "JST PH series connector, B2B-PH-K (http://www.jst-mfg.com/product/pdf/eng/ePH.pdf), generated with kicad-footprint-generator")
-    (tags "connector JST PH side entry")
     (property "Sheetfile" "power.kicad_sch")
     (property "Sheetname" "POWER")
@@
     (property "ki_keywords" "batt voltage-source cell")
     (attr through_hole)
-    (fp_text reference "BT2_1" (at 0.81 5.48) (layer "F.SilkS")
+    (fp_text reference "BT2_1" (at 0 -6.35 unlocked) (layer "F.SilkS")
+        (effects (font (size 1 1) (thickness 0.1)))
+    )
+    (fp_text value "Battery" (at 0 -4.85 unlocked) (layer "F.Fab")
         (effects (font (size 1 1) (thickness 0.15)))
     )
-    (fp_text value "Battery" (at 1 4) (layer "F.Fab")
+    (fp_text user "GND" (at 0.48 2 unlocked) (layer "F.SilkS")
+        (effects (font (size 0.5 0.5) (thickness 0.05)) (justify left bottom))
+    )
+    (fp_text user "+" (at -1.57 1.9 unlocked) (layer "F.SilkS")
+        (effects (font (size 0.5 0.5) (thickness 0.05)) (justify left bottom))
+    )
+    (fp_text user "${REFERENCE}" (at 0 -3.35 unlocked) (layer "F.Fab")
         (effects (font (size 1 1) (thickness 0.15)))
     )
-    (fp_text user "${REFERENCE}" (at 1 1.5) (layer "F.Fab")
-        (effects (font (size 1 1) (thickness 0.15)))
-    )
-    (fp_line (start -2.36 -2.11) (end -2.36 -0.86)
-      (stroke (width 0.12) (type solid)) (layer "F.SilkS"))
-    (fp_line (start -2.06 -1.81) (end -2.06 2.91)
-      (stroke (width 0.12) (type solid)) (layer "F.SilkS"))
-    (fp_line (start -2.06 -0.5) (end -1.45 -0.5)
-      (stroke (width 0.12) (type solid)) (layer "F.SilkS"))
-    (fp_line (start -2.06 0.8) (end -1.45 0.8)
-      (stroke (width 0.12) (type solid)) (layer "F.SilkS"))
-    (fp_line (start -2.06 2.91) (end 4.06 2.91)
-      (stroke (width 0.12) (type solid)) (layer "F.SilkS"))
-    (fp_line (start -1.45 -1.2) (end -1.45 2.3)
-      (stroke (width 0.12) (type solid)) (layer "F.SilkS"))
-    (fp_line (start -1.45 2.3) (end 3.45 2.3)
-      (stroke (width 0.12) (type solid)) (layer "F.SilkS"))
-    (fp_line (start -1.11 -2.11) (end -2.36 -2.11)
-      (stroke (width 0.12) (type solid)) (layer "F.SilkS"))
-    (fp_line (start -0.6 -2.01) (end -0.6 -1.81)
-      (stroke (width 0.12) (type solid)) (layer "F.SilkS"))
-    (fp_line (start -0.3 -2.01) (end -0.6 -2.01)
-      (stroke (width 0.12) (type solid)) (layer "F.SilkS"))
-    (fp_line (start -0.3 -1.91) (end -0.6 -1.91)
-      (stroke (width 0.12) (type solid)) (layer "F.SilkS"))
-    (fp_line (start -0.3 -1.81) (end -0.3 -2.01)
-      (stroke (width 0.12) (type solid)) (layer "F.SilkS"))
-    (fp_line (start 0.5 -1.81) (end 0.5 -1.2)
-      (stroke (width 0.12) (type solid)) (layer "F.SilkS"))
-    (fp_line (start 0.5 -1.2) (end -1.45 -1.2)
-      (stroke (width 0.12) (type solid)) (layer "F.SilkS"))
-    (fp_line (start 0.9 1.8) (end 1.1 1.8)
-      (stroke (width 0.12) (type solid)) (layer "F.SilkS"))
-    (fp_line (start 0.9 2.3) (end 0.9 1.8)
-      (stroke (width 0.12) (type solid)) (layer "F.SilkS"))
-    (fp_line (start 1 2.3) (end 1 1.8)
-      (stroke (width 0.12) (type solid)) (layer "F.SilkS"))
-    (fp_line (start 1.1 1.8) (end 1.1 2.3)
-      (stroke (width 0.12) (type solid)) (layer "F.SilkS"))
-    (fp_line (start 1.5 -1.2) (end 1.5 -1.81)
-      (stroke (width 0.12) (type solid)) (layer "F.SilkS"))
-    (fp_line (start 3.45 -1.2) (end 1.5 -1.2)
-      (stroke (width 0.12) (type solid)) (layer "F.SilkS"))
-    (fp_line (start 3.45 2.3) (end 3.45 -1.2)
-      (stroke (width 0.12) (type solid)) (layer "F.SilkS"))
-    (fp_line (start 4.06 -1.81) (end -2.06 -1.81)
-      (stroke (width 0.12) (type solid)) (layer "F.SilkS"))
-    (fp_line (start 4.06 -0.5) (end 3.45 -0.5)
-      (stroke (width 0.12) (type solid)) (layer "F.SilkS"))
-    (fp_line (start 4.06 0.8) (end 3.45 0.8)
-      (stroke (width 0.12) (type solid)) (layer "F.SilkS"))
-    (fp_line (start 4.06 2.91) (end 4.06 -1.81)
-      (stroke (width 0.12) (type solid)) (layer "F.SilkS"))
-    (fp_line (start -2.45 -2.2) (end -2.45 3.3)
-      (stroke (width 0.05) (type solid)) (layer "F.CrtYd"))
-    (fp_line (start -2.45 3.3) (end 4.45 3.3)
-      (stroke (width 0.05) (type solid)) (layer "F.CrtYd"))
-    (fp_line (start 4.45 -2.2) (end -2.45 -2.2)
-      (stroke (width 0.05) (type solid)) (layer "F.CrtYd"))
-    (fp_line (start 4.45 3.3) (end 4.45 -2.2)
-      (stroke (width 0.05) (type solid)) (layer "F.CrtYd"))
-    (fp_line (start -2.36 -2.11) (end -2.36 -0.86)
-      (stroke (width 0.1) (type solid)) (layer "F.Fab"))
-    (fp_line (start -1.95 -1.7) (end -1.95 2.8)
-      (stroke (width 0.1) (type solid)) (layer "F.Fab"))
-    (fp_line (start -1.95 2.8) (end 3.95 2.8)
-      (stroke (width 0.1) (type solid)) (layer "F.Fab"))
-    (fp_line (start -1.11 -2.11) (end -2.36 -2.11)
-      (stroke (width 0.1) (type solid)) (layer "F.Fab"))
-    (fp_line (start 3.95 -1.7) (end -1.95 -1.7)
-      (stroke (width 0.1) (type solid)) (layer "F.Fab"))
-    (fp_line (start 3.95 2.8) (end 3.95 -1.7)
-      (stroke (width 0.1) (type solid)) (layer "F.Fab"))
-    (pad "1" thru_hole roundrect (at 0 0) (size 1.2 1.75) (drill 0.75) (layers "*.Cu" "*.Mask") (roundrect_rratio 0.208333)
+    (pad "1" thru_hole oval (at -1.27 0) (size 1.7 2.5) (drill 0.762) (layers "*.Cu" "*.Mask")
       (net 58 "Net-(BT2_1-+)") (pinfunction "+") (pintype "passive"))
-    (pad "2" thru_hole oval (at 2 0) (size 1.2 1.75) (drill 0.75) (layers "*.Cu" "*.Mask")
-      (net 6 "GND") (pinfunction "-") (pintype "passive"))
-    (model "${KICAD6_3DMODEL_DIR}/Connector_JST.3dshapes/JST_PH_B2B-PH-K_1x02_P2.00mm_Vertical.wrl"
-      (offset (xyz 0 0 0))
-      (scale (xyz 1 1 1))
-      (rotate (xyz 0 0 0))
-    )
+    (pad "2" thru_hole custom (at 1.27 0) (size 1.7 2.5) (drill 0.762) (layers "*.Cu" "*.Mask")
+      (net 6 "GND") (pinfunction "-") (pintype "passive")
+      (options (clearance outline) (anchor rect))
+      (primitives
+      ))
   )
   (footprint "LED_SMD:LED_0603_1608Metric_Pad1.05x0.95mm_HandSolder" (layer "F.Cu")
